File: Module Boards/Power_Board/Power_Board.kicad_pcb (KiCad board)
At the start: 6 copper layers, 13.8 x 11.6 mm, 30 parts, among them U1 MAX17262REWL+T, U2 MAX77654MENV+T

Commit message: Fixed path dependencies and changed library name to X-MODs
Parts:
- C1, C10, C11, C12, C13, C14, C15, C16, C2: footprint HeepoMind_PcbLib:C0402 -> X-MODs_PcbLib:C0402
- C3, C4, C5, C6, C7, C8, C9: footprint HeepoMind_PcbLib:C0603 -> X-MODs_PcbLib:C0603
- J1: footprint HeepoMind_PcbLib:Power_Board_Castellated_Conn_1.27mm -> X-MODs_PcbLib:Power_Board_Castellated_Conn_1.27mm
- L1: footprint HeepoMind_PcbLib:L0806 -> X-MODs_PcbLib:L0806
- R1, R10, R11, R12, R2, R5, R6, R7, R8, R9: footprint HeepoMind_PcbLib:R0402 -> X-MODs_PcbLib:R0402
- U1: footprint HeepoMind_PcbLib:WLCSP-9_1.468x1.448mm_P0.4mm -> X-MODs_PcbLib:WLCSP-9_1.468x1.448mm_P0.4mm
- U2: footprint HeepoMind_PcbLib:WLCSP-30_2.788x2.338mm_P0.4mm -> X-MODs_PcbLib:WLCSP-30_2.788x2.338mm_P0.4mm
Changed lines of the file:
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@@
 	(net 29 "/[2] PMIC/IN_LDO1")
 	(net 30 "unconnected-(U2-TBIAS-PadD3)")
-	(footprint "HeepoMind_PcbLib:C0603"
+	(footprint "X-MODs_PcbLib:C0603"
 		(layer "F.Cu")
 		(at 142.4975 99.2325 180)
@@
 			)
 		)
-		(property "Footprint" "HeepoMind_PcbLib:C0603"
+		(property "Footprint" "X-MODs_PcbLib:C0603"
 			(at 0 -9 180)
 			(unlocked yes)
@@
 		)
 	)
-	(footprint "HeepoMind_PcbLib:C0402"
+	(footprint "X-MODs_PcbLib:C0402"
 		(layer "F.Cu")
 		(at 141.7725 103.9325)
@@
 			)
 		)
-		(property "Footprint" "HeepoMind_PcbLib:C0402"
+		(property "Footprint" "X-MODs_PcbLib:C0402"
 			(at 0 -9 0)
 			(unlocked yes)
@@
 		)
 	)
-	(footprint "HeepoMind_PcbLib:R0402"
+	(footprint "X-MODs_PcbLib:R0402"
 		(layer "F.Cu")
 		(at 142.1225 96.4325 90)
@@
 			)
 		)
-		(property "Footprint" "HeepoMind_PcbLib:R0402"
+		(property "Footprint" "X-MODs_PcbLib:R0402"
 			(at 0 -9 90)
 			(unlocked yes)
@@
 		)
 	)
-	(footprint "HeepoMind_PcbLib:C0603"
+	(footprint "X-MODs_PcbLib:C0603"
 		(layer "F.Cu")
 		(at 150.0475 101.1325)
@@
 			)
 		)
-		(property "Footprint" "HeepoMind_PcbLib:C0603"
+		(property "Footprint" "X-MODs_PcbLib:C0603"
 			(at 0 -9 0)
 			(unlocked yes)
@@
 		)
 	)
-	(footprint "HeepoMind_PcbLib:C0402"
+	(footprint "X-MODs_PcbLib:C0402"
 		(layer "F.Cu")
 		(at 145.4725 96.4325 90)
@@
 			)
 		)
-		(property "Footprint" "HeepoMind_PcbLib:C0402"
+		(property "Footprint" "X-MODs_PcbLib:C0402"
 			(at 0 -9 90)
 			(unlocked yes)
@@
 		)
 	)
-	(footprint "HeepoMind_PcbLib:C0603"
+	(footprint "X-MODs_PcbLib:C0603"
 		(layer "F.Cu")
 		(at 150.0475 98.3325)
@@
 			)
 		)
-		(property "Footprint" "HeepoMind_PcbLib:C0603"
+		(property "Footprint" "X-MODs_PcbLib:C0603"
 			(at 0 -9 0)
 			(unlocked yes)
@@
 		)
 	)
-	(footprint "HeepoMind_PcbLib:R0402"
+	(footprint "X-MODs_PcbLib:R0402"
 		(layer "F.Cu")
 		(at 150.8475 96.4325 -90)
@@
 			)
 		)
-		(property "Footprint" "HeepoMind_PcbLib:R0402"
+		(property "Footprint" "X-MODs_PcbLib:R0402"
 			(at 0 -9 -90)
 			(unlocked yes)
@@
 		)
 	)
-	(footprint "HeepoMind_PcbLib:C0402"
+	(footprint "X-MODs_PcbLib:C0402"
 		(layer "F.Cu")
 		(at 142.9975 98.1575 180)
@@
 			)
 		)
-		(property "Footprint" "HeepoMind_PcbLib:C0402"
+		(property "Footprint" "X-MODs_PcbLib:C0402"
 			(at 0 -9 180)
 			(unlocked yes)
@@
 		)
 	)
-	(footprint "HeepoMind_PcbLib:C0402"
+	(footprint "X-MODs_PcbLib:C0402"
 		(layer "F.Cu")
 		(at 147.3225 96.4325 90)
@@
 			)
 		)
-		(property "Footprint" "HeepoMind_PcbLib:C0402"
+		(property "Footprint" "X-MODs_PcbLib:C0402"
 			(at 0 -9 90)
 			(unlocked yes)
@@
 		)
 	)
-	(footprint "HeepoMind_PcbLib:R0402"
+	(footprint "X-MODs_PcbLib:R0402"
 		(layer "F.Cu")
 		(at 151.6725 103.6325 90)
@@
 			)
 		)
-		(property "Footprint" "HeepoMind_PcbLib:R0402"
+		(property "Footprint" "X-MODs_PcbLib:R0402"
 			(at 0 -9 90)
 			(unlocked yes)
@@
 		)
 	)
-	(footprint "HeepoMind_PcbLib:C0402"
+	(footprint "X-MODs_PcbLib:C0402"
 		(layer "F.Cu")
 		(at 141.7725 101.3575)
@@
 			)
 		)
-		(property "Footprint" "HeepoMind_PcbLib:C0402"
+		(property "Footprint" "X-MODs_PcbLib:C0402"
 			(at 0 -9 0)
 			(unlocked yes)
@@
 		)
 	)
-	(footprint "HeepoMind_PcbLib:C0402"
+	(footprint "X-MODs_PcbLib:C0402"
 		(layer "F.Cu")
 		(at 149.1975 96.4325 90)
@@
 			)
 		)
-		(property "Footprint" "HeepoMind_PcbLib:C0402"
+		(property "Footprint" "X-MODs_PcbLib:C0402"
 			(at 0 -9 90)
 			(unlocked yes)
@@
 		)
 	)
-	(footprint "HeepoMind_PcbLib:L0806"
+	(footprint "X-MODs_PcbLib:L0806"
 		(layer "F.Cu")
 		(at 146.9475 103.4825 180)
@@
 			)
 		)
-		(property "Footprint" "HeepoMind_PcbLib:L0806"
+		(property "Footprint" "X-MODs_PcbLib:L0806"
 			(at 0 -9 180)
 			(unlocked yes)
@@
 		)
 	)
-	(footprint "HeepoMind_PcbLib:R0402"
+	(footprint "X-MODs_PcbLib:R0402"
 		(layer "F.Cu")
 		(at 150.8475 103.6325 90)
@@
 			)
 		)
-		(property "Footprint" "HeepoMind_PcbLib:R0402"
+		(property "Footprint" "X-MODs_PcbLib:R0402"
 			(at 0 -9 90)
 			(unlocked yes)
@@
 		)
 	)
-	(footprint "HeepoMind_PcbLib:C0402"
+	(footprint "X-MODs_PcbLib:C0402"
 		(layer "F.Cu")
 		(at 148.2475 96.4325 90)
@@
 			)
 		)
-		(property "Footprint" "HeepoMind_PcbLib:C0402"
+		(property "Footprint" "X-MODs_PcbLib:C0402"
 			(at 0 -9 90)
 			(unlocked yes)
@@
 		)
 	)
-	(footprint "HeepoMind_PcbLib:C0402"
+	(footprint "X-MODs_PcbLib:C0402"
 		(layer "F.Cu")
 		(at 148.6725 103.4825 90)
@@
 			)
 		)
-		(property "Footprint" "HeepoMind_PcbLib:C0402"
+		(property "Footprint" "X-MODs_PcbLib:C0402"
 			(at 0 -9 90)
 			(unlocked yes)
@@
 		)
 	)
-	(footprint "HeepoMind_PcbLib:R0402"
+	(footprint "X-MODs_PcbLib:R0402"
 		(layer "F.Cu")
 		(at 151.6725 96.4325 -90)
@@
 			)
 		)
-		(property "Footprint" "HeepoMind_PcbLib:R0402"
+		(property "Footprint" "X-MODs_PcbLib:R0402"
 			(at 0 -9 -90)
 			(unlocked yes)
@@
 		)
 	)
-	(footprint "HeepoMind_PcbLib:C0603"
+	(footprint "X-MODs_PcbLib:C0603"
 		(layer "F.Cu")
 		(at 143.4975 102.2325 -90)
@@
 			)
 		)
-		(property "Footprint" "HeepoMind_PcbLib:C0603"
+		(property "Footprint" "X-MODs_PcbLib:C0603"
 			(at 0 -9 -90)
 			(unlocked yes)
@@
 		)
 	)
-	(footprint "HeepoMind_PcbLib:WLCSP-30_2.788x2.338mm_P0.4mm"
+	(footprint "X-MODs_PcbLib:WLCSP-30_2.788x2.338mm_P0.4mm"
 		(layer "F.Cu")
 		(at 146.0725 98.9325)
@@
 			)
 		)
-		(property "Footprint" "HeepoMind_PcbLib:WLCSP-30_2.788x2.338mm_P0.4mm"
+		(property "Footprint" "X-MODs_PcbLib:WLCSP-30_2.788x2.338mm_P0.4mm"
 			(at 0 -9 0)
 			(unlocked yes)
@@
 			(layers "F.Cu" "F.Paste" "F.Mask")
 			(net 26 "nRST")
-			(pinfunction "nRST")
+			(pinfunction "~{RST}")
 			(pintype "passive")
 			(solder_paste_margin_ratio -1)
@@
 			(layers "F.Cu" "F.Paste" "F.Mask")
 			(net 25 "nIRQ")
-			(pinfunction "nIRQ")
+			(pinfunction "~{IRQ}")
 			(pintype "passive")
 			(solder_paste_margin_ratio -1)
@@
 			(layers "F.Cu" "F.Paste" "F.Mask")
 			(net 24 "nEN")
-			(pinfunction "nEN")
+			(pinfunction "~{EN}")
 			(pintype "passive")
 			(solder_paste_margin_ratio -1)
@@
 		)
 	)
-	(footprint "HeepoMind_PcbLib:C0603"
+	(footprint "X-MODs_PcbLib:C0603"
 		(layer "F.Cu")
 		(at 150.0475 99.7325)
@@
 			)
 		)
-		(property "Footprint" "HeepoMind_PcbLib:C0603"
+		(property "Footprint" "X-MODs_PcbLib:C0603"
 			(at 0 -9 0)
 			(unlocked yes)
@@
 		)
 	)
-	(footprint "HeepoMind_PcbLib:WLCSP-9_1.468x1.448mm_P0.4mm"
+	(footprint "X-MODs_PcbLib:WLCSP-9_1.468x1.448mm_P0.4mm"
 		(layer "F.Cu")
 		(at 141.7725 102.6575)
@@
 			)
 		)
-		(property "Footprint" "HeepoMind_PcbLib:WLCSP-9_1.468x1.448mm_P0.4mm"
+		(property "Footprint" "X-MODs_PcbLib:WLCSP-9_1.468x1.448mm_P0.4mm"
 			(at 0 -9 0)
 			(unlocked yes)
@@
 		)
 	)
-	(footprint "HeepoMind_PcbLib:R0402"
+	(footprint "X-MODs_PcbLib:R0402"
 		(layer "F.Cu")
 		(at 144.6475 96.4325 -90)
@@
 			)
 		)
-		(property "Footprint" "HeepoMind_PcbLib:R0402"
+		(property "Footprint" "X-MODs_PcbLib:R0402"
 			(at 0 -9 -90)
 			(unlocked yes)
@@
 		)
 	)
-	(footprint "HeepoMind_PcbLib:C0603"
+	(footprint "X-MODs_PcbLib:C0603"
 		(layer "F.Cu")
 		(at 147.0725 101.4325)
@@
 			)
 		)
-		(property "Footprint" "HeepoMind_PcbLib:C0603"
+		(property "Footprint" "X-MODs_PcbLib:C0603"
 			(at 0 -9 0)
 			(unlocked yes)
@@
 		)
 	)
-	(footprint "HeepoMind_PcbLib:R0402"
+	(footprint "X-MODs_PcbLib:R0402"
 		(layer "F.Cu")
 		(at 141.2925 96.4325 90)
@@
 			)
 		)
-		(property "Footprint" "HeepoMind_PcbLib:R0402"
+		(property "Footprint" "X-MODs_PcbLib:R0402"
 			(at 0 -9 90)
 			(unlocked yes)
@@
 		)
 	)
-	(footprint "HeepoMind_PcbLib:C0603"
+	(footprint "X-MODs_PcbLib:C0603"
 		(layer "F.Cu")
 		(at 144.8475 102.2325 -90)
@@
 			)
 		)
-		(property "Footprint" "HeepoMind_PcbLib:C0603"
+		(property "Footprint" "X-MODs_PcbLib:C0603"
 			(at 0 -9 -90)
 			(unlocked yes)
@@
 		)
 	)
-	(footprint "HeepoMind_PcbLib:R0402"
+	(footprint "X-MODs_PcbLib:R0402"
 		(layer "F.Cu")
 		(at 150.0225 103.6325 90)
@@
 			)
 		)
-		(property "Footprint" "HeepoMind_PcbLib:R0402"
+		(property "Footprint" "X-MODs_PcbLib:R0402"
 			(at 0 -9 90)
 			(unlocked yes)
@@
 		)
 	)
-	(footprint "HeepoMind_PcbLib:Power_Board_Castellated_Conn_1.27mm"
+	(footprint "X-MODs_PcbLib:Power_Board_Castellated_Conn_1.27mm"
 		(layer "F.Cu")
 		(at 146.485 100.02)
@@
 			)
 		)
-		(property "Footprint" "HeepoMind_PcbLib:Power_Board_Castellated_Conn_1.27mm"
+		(property "Footprint" "X-MODs_PcbLib:Power_Board_Castellated_Conn_1.27mm"
 			(at 0 -9 0)
 			(unlocked yes)
@@
 		)
 	)
-	(footprint "HeepoMind_PcbLib:C0402"
+	(footprint "X-MODs_PcbLib:C0402"
 		(layer "F.Cu")
 		(at 146.3975 96.4325 90)
@@
 			)
 		)
-		(property "Footprint" "HeepoMind_PcbLib:C0402"
+		(property "Footprint" "X-MODs_PcbLib:C0402"
 			(at 0 -9 90)
 			(unlocked yes)
@@
 		)
 	)
-	(footprint "HeepoMind_PcbLib:R0402"
+	(footprint "X-MODs_PcbLib:R0402"
 		(layer "F.Cu")
 		(at 150.0225 96.4325 -90)
@@
 			)
 		)
-		(property "Footprint" "HeepoMind_PcbLib:R0402"
+		(property "Footprint" "X-MODs_PcbLib:R0402"
 			(at 0 -9 -90)
 			(unlocked yes)
@@
 		)
 	)
-	(footprint "HeepoMind_PcbLib:R0402"
+	(footprint "X-MODs_PcbLib:R0402"
 		(layer "F.Cu")
 		(at 143.8225 96.4325 -90)
@@
 			)
 		)
-		(property "Footprint" "HeepoMind_PcbLib:R0402"
+		(property "Footprint" "X-MODs_PcbLib:R0402"
 			(at 0 -9 -90)
 			(unlocked yes)
