File: Module Boards/Power_Board/[1] Battery Gauge & Connectors.kicad_sch (KiCad schematic)
At the start: 6 parts, among them U1 MAX17262REWL+T

Commit message: Fixed path dependencies and changed library name to X-MODs
Parts:
- C1: footprint HeepoMind_PcbLib:C0402 -> X-MODs_PcbLib:C0402; symbol HeepoMind_SchLib:GRM155R71A104JA01D -> X-MODs_SchLib:GRM155R71A104JA01D
- C2: footprint HeepoMind_PcbLib:C0402 -> X-MODs_PcbLib:C0402; symbol HeepoMind_SchLib:GRM155R60J474KE19 -> X-MODs_SchLib:GRM155R60J474KE19
- J1: footprint HeepoMind_PcbLib:Power_Board_Castellated_Conn_1.27mm -> X-MODs_PcbLib:Power_Board_Castellated_Conn_1.27mm; symbol HeepoMind_SchLib:Power_Board_Castellated_Conn_1.27mm -> X-MODs_SchLib:Power_Board_Castellated_Conn_1.27mm
- R1: footprint HeepoMind_PcbLib:R0402 -> X-MODs_PcbLib:R0402; symbol HeepoMind_SchLib:R -> X-MODs_SchLib:R
- R2: footprint HeepoMind_PcbLib:R0402 -> X-MODs_PcbLib:R0402; symbol HeepoMind_SchLib:RK73Z1ETTP -> X-MODs_SchLib:RK73Z1ETTP
- U1: footprint HeepoMind_PcbLib:WLCSP-9_1.468x1.448mm_P0.4mm -> X-MODs_PcbLib:WLCSP-9_1.468x1.448mm_P0.4mm; symbol HeepoMind_SchLib:MAX17262REWL+T -> X-MODs_SchLib:MAX17262REWL+T
Changed lines of the file:
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@@
 	)
 	(symbol
-		(lib_id "HeepoMind_SchLib:RK73Z1ETTP")
+		(lib_id "X-MODs_SchLib:RK73Z1ETTP")
 		(at 118.11 113.03 270)
 		(unit 1)
@@
 			)
 		)
-		(property "Footprint" "HeepoMind_PcbLib:R0402"
+		(property "Footprint" "X-MODs_PcbLib:R0402"
 			(at 114.808 98.044 0)
 			(effects
@@
 	)
 	(symbol
-		(lib_id "HeepoMind_SchLib:GRM155R71A104JA01D")
+		(lib_id "X-MODs_SchLib:GRM155R71A104JA01D")
 		(at 48.26 96.52 270)
 		(unit 1)
@@
 			)
 		)
-		(property "Footprint" "HeepoMind_PcbLib:C0402"
+		(property "Footprint" "X-MODs_PcbLib:C0402"
 			(at 39.624 59.436 0)
 			(effects
@@
 	)
 	(symbol
-		(lib_id "HeepoMind_SchLib:Power_Board_Castellated_Conn_1.27mm")
+		(lib_id "X-MODs_SchLib:Power_Board_Castellated_Conn_1.27mm")
 		(at 243.84 59.69 0)
 		(unit 3)
@@
 			)
 		)
-		(property "Footprint" "HeepoMind_PcbLib:Power_Board_Castellated_Conn_1.27mm"
+		(property "Footprint" "X-MODs_PcbLib:Power_Board_Castellated_Conn_1.27mm"
 			(at 252.984 90.17 0)
 			(effects
@@
 	)
 	(symbol
-		(lib_id "HeepoMind_SchLib:Power_Board_Castellated_Conn_1.27mm")
+		(lib_id "X-MODs_SchLib:Power_Board_Castellated_Conn_1.27mm")
 		(at 201.93 59.69 0)
 		(unit 1)
@@
 			)
 		)
-		(property "Footprint" "HeepoMind_PcbLib:Power_Board_Castellated_Conn_1.27mm"
+		(property "Footprint" "X-MODs_PcbLib:Power_Board_Castellated_Conn_1.27mm"
 			(at 211.074 90.17 0)
 			(effects
@@
 	)
 	(symbol
-		(lib_id "HeepoMind_SchLib:Power_Board_Castellated_Conn_1.27mm")
+		(lib_id "X-MODs_SchLib:Power_Board_Castellated_Conn_1.27mm")
 		(at 201.93 99.06 0)
 		(unit 2)
@@
 			)
 		)
-		(property "Footprint" "HeepoMind_PcbLib:Power_Board_Castellated_Conn_1.27mm"
+		(property "Footprint" "X-MODs_PcbLib:Power_Board_Castellated_Conn_1.27mm"
 			(at 211.074 129.54 0)
 			(effects
@@
 	)
 	(symbol
-		(lib_id "HeepoMind_SchLib:GRM155R60J474KE19")
+		(lib_id "X-MODs_SchLib:GRM155R60J474KE19")
 		(at 99.06 115.57 270)
 		(unit 1)
@@
 			)
 		)
-		(property "Footprint" "HeepoMind_PcbLib:C0402"
+		(property "Footprint" "X-MODs_PcbLib:C0402"
 			(at 90.932 89.154 0)
 			(effects
@@
 	)
 	(symbol
-		(lib_id "HeepoMind_SchLib:MAX17262REWL+T")
+		(lib_id "X-MODs_SchLib:MAX17262REWL+T")
 		(at 71.12 87.63 0)
 		(unit 1)
@@
 			)
 		)
-		(property "Footprint" "HeepoMind_PcbLib:WLCSP-9_1.468x1.448mm_P0.4mm"
+		(property "Footprint" "X-MODs_PcbLib:WLCSP-9_1.468x1.448mm_P0.4mm"
 			(at 70.866 122.936 0)
 			(effects
@@
 	)
 	(symbol
-		(lib_id "HeepoMind_SchLib:R")
+		(lib_id "X-MODs_SchLib:R")
 		(at 118.11 95.25 90)
 		(unit 1)
@@
 			)
 		)
-		(property "Footprint" "HeepoMind_PcbLib:R0402"
+		(property "Footprint" "X-MODs_PcbLib:R0402"
 			(at 121.412 95.25 0)
 			(effects
@@
 	)
 	(symbol
-		(lib_id "HeepoMind_SchLib:Power_Board_Castellated_Conn_1.27mm")
+		(lib_id "X-MODs_SchLib:Power_Board_Castellated_Conn_1.27mm")
 		(at 243.84 99.06 0)
 		(unit 4)
@@
 			)
 		)
-		(property "Footprint" "HeepoMind_PcbLib:Power_Board_Castellated_Conn_1.27mm"
+		(property "Footprint" "X-MODs_PcbLib:Power_Board_Castellated_Conn_1.27mm"
 			(at 252.984 129.54 0)
 			(effects
