File: Module Boards/Power_Board/[2] PMIC.kicad_sch (KiCad schematic)
At the start: 24 parts, among them U2 MAX77654MENV+T

Commit message: Fixed path dependencies and changed library name to X-MODs
Parts:
- C10: footprint HeepoMind_PcbLib:C0402 -> X-MODs_PcbLib:C0402; symbol HeepoMind_SchLib:GRM15XR71C332KA86D -> X-MODs_SchLib:GRM15XR71C332KA86D
- C11, C14, C15, C16: footprint HeepoMind_PcbLib:C0402 -> X-MODs_PcbLib:C0402; symbol HeepoMind_SchLib:C0402C105K8PACTU -> X-MODs_SchLib:C0402C105K8PACTU
- C12, C13: footprint HeepoMind_PcbLib:C0402 -> X-MODs_PcbLib:C0402; symbol HeepoMind_SchLib:GRM155R61C225KE44D -> X-MODs_SchLib:GRM155R61C225KE44D
- C3, C4: footprint HeepoMind_PcbLib:C0603 -> X-MODs_PcbLib:C0603; symbol HeepoMind_SchLib:GRM188R61E475KE11D -> X-MODs_SchLib:GRM188R61E475KE11D
- C5, C6, C7, C8, C9: footprint HeepoMind_PcbLib:C0603 -> X-MODs_PcbLib:C0603; symbol HeepoMind_SchLib:GRM188R61A226ME15D -> X-MODs_SchLib:GRM188R61A226ME15D
- L1: footprint HeepoMind_PcbLib:L0806 -> X-MODs_PcbLib:L0806; symbol HeepoMind_SchLib:DFE201612E-1R5M=P2 -> X-MODs_SchLib:DFE201612E-1R5M=P2
- R10, R11, R12, R5, R6, R7: footprint HeepoMind_PcbLib:R0402 -> X-MODs_PcbLib:R0402; symbol HeepoMind_SchLib:RK73Z1ETTP -> X-MODs_SchLib:RK73Z1ETTP
- R8, R9: footprint HeepoMind_PcbLib:R0402 -> X-MODs_PcbLib:R0402; symbol HeepoMind_SchLib:CRCW0402100KFKEDC -> X-MODs_SchLib:CRCW0402100KFKEDC
- U2: footprint HeepoMind_PcbLib:WLCSP-30_2.788x2.338mm_P0.4mm -> X-MODs_PcbLib:WLCSP-30_2.788x2.338mm_P0.4mm; symbol HeepoMind_SchLib:MAX77654MENV+T -> X-MODs_SchLib:MAX77654MENV+T
Changed lines of the file:
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@@
 	)
 	(symbol
-		(lib_id "HeepoMind_SchLib:GRM188R61E475KE11D")
+		(lib_id "X-MODs_SchLib:GRM188R61E475KE11D")
 		(at 55.88 67.31 270)
 		(unit 1)
@@
 			)
 		)
-		(property "Footprint" "HeepoMind_PcbLib:C0603"
+		(property "Footprint" "X-MODs_PcbLib:C0603"
 			(at 47.752 40.894 0)
 			(effects
@@
 	)
 	(symbol
-		(lib_id "HeepoMind_SchLib:C0402C105K8PACTU")
+		(lib_id "X-MODs_SchLib:C0402C105K8PACTU")
 		(at 81.28 113.03 270)
 		(unit 1)
@@
 			)
 		)
-		(property "Footprint" "HeepoMind_PcbLib:C0402"
+		(property "Footprint" "X-MODs_PcbLib:C0402"
 			(at 72.644 91.186 0)
 			(effects
@@
 	)
 	(symbol
-		(lib_id "HeepoMind_SchLib:RK73Z1ETTP")
+		(lib_id "X-MODs_SchLib:RK73Z1ETTP")
 		(at 240.03 73.66 270)
 		(unit 1)
@@
 			)
 		)
-		(property "Footprint" "HeepoMind_PcbLib:R0402"
+		(property "Footprint" "X-MODs_PcbLib:R0402"
 			(at 236.728 58.674 0)
 			(effects
@@
 	)
 	(symbol
-		(lib_id "HeepoMind_SchLib:CRCW0402100KFKEDC")
+		(lib_id "X-MODs_SchLib:CRCW0402100KFKEDC")
 		(at 218.44 116.84 90)
 		(unit 1)
@@
 			)
 		)
-		(property "Footprint" "HeepoMind_PcbLib:R0402"
+		(property "Footprint" "X-MODs_PcbLib:R0402"
 			(at 221.742 131.826 0)
 			(effects
@@
 	)
 	(symbol
-		(lib_id "HeepoMind_SchLib:MAX77654MENV+T")
+		(lib_id "X-MODs_SchLib:MAX77654MENV+T")
 		(at 99.06 50.8 0)
 		(unit 1)
@@
 			)
 		)
-		(property "Footprint" "HeepoMind_PcbLib:WLCSP-30_2.788x2.338mm_P0.4mm"
+		(property "Footprint" "X-MODs_PcbLib:WLCSP-30_2.788x2.338mm_P0.4mm"
 			(at 125.222 150.368 0)
 			(effects
@@
 	)
 	(symbol
-		(lib_id "HeepoMind_SchLib:C0402C105K8PACTU")
+		(lib_id "X-MODs_SchLib:C0402C105K8PACTU")
 		(at 172.72 109.22 270)
 		(unit 1)
@@
 			)
 		)
-		(property "Footprint" "HeepoMind_PcbLib:C0402"
+		(property "Footprint" "X-MODs_PcbLib:C0402"
 			(at 164.084 87.376 0)
 			(effects
@@
 	)
 	(symbol
-		(lib_id "HeepoMind_SchLib:GRM188R61A226ME15D")
+		(lib_id "X-MODs_SchLib:GRM188R61A226ME15D")
 		(at 184.15 73.66 270)
 		(unit 1)
@@
 			)
 		)
-		(property "Footprint" "HeepoMind_PcbLib:C0603"
+		(property "Footprint" "X-MODs_PcbLib:C0603"
 			(at 176.022 48.26 0)
 			(effects
@@
 	)
 	(symbol
-		(lib_id "HeepoMind_SchLib:GRM15XR71C332KA86D")
+		(lib_id "X-MODs_SchLib:GRM15XR71C332KA86D")
 		(at 81.28 92.71 0)
 		(unit 1)
@@
 			)
 		)
-		(property "Footprint" "HeepoMind_PcbLib:C0402"
+		(property "Footprint" "X-MODs_PcbLib:C0402"
 			(at 55.88 100.838 0)
 			(effects
@@
 	)
 	(symbol
-		(lib_id "HeepoMind_SchLib:GRM188R61E475KE11D")
+		(lib_id "X-MODs_SchLib:GRM188R61E475KE11D")
 		(at 31.75 59.69 270)
 		(unit 1)
@@
 			)
 		)
-		(property "Footprint" "HeepoMind_PcbLib:C0603"
+		(property "Footprint" "X-MODs_PcbLib:C0603"
 			(at 23.622 33.274 0)
 			(effects
@@
 	)
 	(symbol
-		(lib_id "HeepoMind_SchLib:RK73Z1ETTP")
+		(lib_id "X-MODs_SchLib:RK73Z1ETTP")
 		(at 207.01 73.66 270)
 		(unit 1)
@@
 			)
 		)
-		(property "Footprint" "HeepoMind_PcbLib:R0402"
+		(property "Footprint" "X-MODs_PcbLib:R0402"
 			(at 203.708 58.674 0)
 			(effects
@@
 	)
 	(symbol
-		(lib_id "HeepoMind_SchLib:C0402C105K8PACTU")
+		(lib_id "X-MODs_SchLib:C0402C105K8PACTU")
 		(at 184.15 110.49 270)
 		(unit 1)
@@
 			)
 		)
-		(property "Footprint" "HeepoMind_PcbLib:C0402"
+		(property "Footprint" "X-MODs_PcbLib:C0402"
 			(at 175.514 88.646 0)
 			(effects
@@
 	)
 	(symbol
-		(lib_id "HeepoMind_SchLib:CRCW0402100KFKEDC")
+		(lib_id "X-MODs_SchLib:CRCW0402100KFKEDC")
 		(at 228.6 116.84 90)
 		(unit 1)
@@
 			)
 		)
-		(property "Footprint" "HeepoMind_PcbLib:R0402"
+		(property "Footprint" "X-MODs_PcbLib:R0402"
 			(at 231.902 131.826 0)
 			(effects
@@
 	)
 	(symbol
-		(lib_id "HeepoMind_SchLib:DFE201612E-1R5M=P2")
+		(lib_id "X-MODs_SchLib:DFE201612E-1R5M=P2")
 		(at 81.28 80.01 0)
 		(unit 1)
@@
 			)
 		)
-		(property "Footprint" "HeepoMind_PcbLib:L0806"
+		(property "Footprint" "X-MODs_PcbLib:L0806"
 			(at 66.294 83.312 0)
 			(effects
@@
 	)
 	(symbol
-		(lib_id "HeepoMind_SchLib:GRM155R61C225KE44D")
+		(lib_id "X-MODs_SchLib:GRM155R61C225KE44D")
 		(at 161.29 109.22 270)
 		(unit 1)
@@
 			)
 		)
-		(property "Footprint" "HeepoMind_PcbLib:C0402"
+		(property "Footprint" "X-MODs_PcbLib:C0402"
 			(at 153.162 84.074 0)
 			(effects
@@
 	)
 	(symbol
-		(lib_id "HeepoMind_SchLib:GRM155R61C225KE44D")
+		(lib_id "X-MODs_SchLib:GRM155R61C225KE44D")
 		(at 149.86 109.22 270)
 		(unit 1)
@@
 			)
 		)
-		(property "Footprint" "HeepoMind_PcbLib:C0402"
+		(property "Footprint" "X-MODs_PcbLib:C0402"
 			(at 141.732 84.074 0)
 			(effects
@@
 	)
 	(symbol
-		(lib_id "HeepoMind_SchLib:RK73Z1ETTP")
+		(lib_id "X-MODs_SchLib:RK73Z1ETTP")
 		(at 195.58 73.66 270)
 		(unit 1)
@@
 			)
 		)
-		(property "Footprint" "HeepoMind_PcbLib:R0402"
+		(property "Footprint" "X-MODs_PcbLib:R0402"
 			(at 192.278 58.674 0)
 			(effects
@@
 	)
 	(symbol
-		(lib_id "HeepoMind_SchLib:RK73Z1ETTP")
+		(lib_id "X-MODs_SchLib:RK73Z1ETTP")
 		(at 218.44 73.66 270)
 		(unit 1)
@@
 			)
 		)
-		(property "Footprint" "HeepoMind_PcbLib:R0402"
+		(property "Footprint" "X-MODs_PcbLib:R0402"
 			(at 215.138 58.674 0)
 			(effects
@@
 	)
 	(symbol
-		(lib_id "HeepoMind_SchLib:RK73Z1ETTP")
+		(lib_id "X-MODs_SchLib:RK73Z1ETTP")
 		(at 228.6 73.66 270)
 		(unit 1)
@@
 			)
 		)
-		(property "Footprint" "HeepoMind_PcbLib:R0402"
+		(property "Footprint" "X-MODs_PcbLib:R0402"
 			(at 225.298 58.674 0)
 			(effects
@@
 	)
 	(symbol
-		(lib_id "HeepoMind_SchLib:C0402C105K8PACTU")
+		(lib_id "X-MODs_SchLib:C0402C105K8PACTU")
 		(at 69.85 105.41 270)
 		(unit 1)
@@
 			)
 		)
-		(property "Footprint" "HeepoMind_PcbLib:C0402"
+		(property "Footprint" "X-MODs_PcbLib:C0402"
 			(at 61.214 83.566 0)
 			(effects
@@
 	)
 	(symbol
-		(lib_id "HeepoMind_SchLib:RK73Z1ETTP")
+		(lib_id "X-MODs_SchLib:RK73Z1ETTP")
 		(at 251.46 73.66 270)
 		(unit 1)
@@
 			)
 		)
-		(property "Footprint" "HeepoMind_PcbLib:R0402"
+		(property "Footprint" "X-MODs_PcbLib:R0402"
 			(at 248.158 58.674 0)
 			(effects
@@
 	)
 	(symbol
-		(lib_id "HeepoMind_SchLib:GRM188R61A226ME15D")
+		(lib_id "X-MODs_SchLib:GRM188R61A226ME15D")
 		(at 161.29 73.66 270)
 		(unit 1)
@@
 			)
 		)
-		(property "Footprint" "HeepoMind_PcbLib:C0603"
+		(property "Footprint" "X-MODs_PcbLib:C0603"
 			(at 153.162 48.26 0)
 			(effects
@@
 	)
 	(symbol
-		(lib_id "HeepoMind_SchLib:GRM188R61A226ME15D")
+		(lib_id "X-MODs_SchLib:GRM188R61A226ME15D")
 		(at 138.43 73.66 270)
 		(unit 1)
@@
 			)
 		)
-		(property "Footprint" "HeepoMind_PcbLib:C0603"
+		(property "Footprint" "X-MODs_PcbLib:C0603"
 			(at 130.302 48.26 0)
 			(effects
@@
 	)
 	(symbol
-		(lib_id "HeepoMind_SchLib:GRM188R61A226ME15D")
+		(lib_id "X-MODs_SchLib:GRM188R61A226ME15D")
 		(at 172.72 73.66 270)
 		(unit 1)
@@
 			)
 		)
-		(property "Footprint" "HeepoMind_PcbLib:C0603"
+		(property "Footprint" "X-MODs_PcbLib:C0603"
 			(at 164.592 48.26 0)
 			(effects
@@
 	)
 	(symbol
-		(lib_id "HeepoMind_SchLib:GRM188R61A226ME15D")
+		(lib_id "X-MODs_SchLib:GRM188R61A226ME15D")
 		(at 149.86 73.66 270)
 		(unit 1)
@@
 			)
 		)
-		(property "Footprint" "HeepoMind_PcbLib:C0603"
+		(property "Footprint" "X-MODs_PcbLib:C0603"
 			(at 141.732 48.26 0)
 			(effects
