File: Socket Boards/Power_Board_Socket/[1] 1.27 mm Flexypin to 2.54 mm Header Adapter.kicad_sch (KiCad schematic)
At the start: 2 parts

Commit message: Fixed paths of module boards
Parts:
- J1: footprint HeepoMind_PcbLib:Power_Board_Socket_Conn_1.27mm -> X-MODs_PcbLib:Power_Board_Socket_Conn_1.27mm; symbol HeepoMind_SchLib:Power_Board_Socket_Conn_1.27mm -> X-MODs_SchLib:Power_Board_Socket_Conn_1.27mm
- J2: footprint HeepoMind_PcbLib:Power_Board_Header_Conn_2.54mm -> X-MODs_PcbLib:Power_Board_Header_Conn_2.54mm; symbol HeepoMind_SchLib:Power_Board_Header_Conn_2.54mm -> X-MODs_SchLib:Power_Board_Header_Conn_2.54mm
Changed lines of the file:
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@@
 	)
 	(symbol
-		(lib_id "HeepoMind_SchLib:Power_Board_Socket_Conn_1.27mm")
+		(lib_id "X-MODs_SchLib:Power_Board_Socket_Conn_1.27mm")
 		(at 99.06 114.3 0)
 		(mirror y)
@@
 			)
 		)
-		(property "Footprint" "HeepoMind_PcbLib:Power_Board_Socket_Conn_1.27mm"
-			(at 89.916 144.78 0)
+		(property "Footprint" "X-MODs_PcbLib:Power_Board_Socket_Conn_1.27mm"
+			(at 90.932 146.05 0)
 			(effects
 				(font
@@
 		)
 		(property "Description" "Power_Board_Socket_Conn_1.27mm"
-			(at 101.092 142.748 0)
+			(at 99.822 144.018 0)
 			(effects
 				(font
@@
 	)
 	(symbol
-		(lib_id "HeepoMind_SchLib:Power_Board_Header_Conn_2.54mm")
+		(lib_id "X-MODs_SchLib:Power_Board_Header_Conn_2.54mm")
 		(at 132.08 66.04 0)
 		(unit 1)
@@
 			)
 		)
-		(property "Footprint" "HeepoMind_PcbLib:Power_Board_Header_Conn_2.54mm"
-			(at 132.842 64.77 0)
+		(property "Footprint" "X-MODs_PcbLib:Power_Board_Header_Conn_2.54mm"
+			(at 133.858 122.936 0)
 			(effects
 				(font
@@
 	)
 	(symbol
-		(lib_id "HeepoMind_SchLib:Power_Board_Socket_Conn_1.27mm")
+		(lib_id "X-MODs_SchLib:Power_Board_Socket_Conn_1.27mm")
 		(at 99.06 45.72 0)
 		(mirror y)
@@
 			)
 		)
-		(property "Footprint" "HeepoMind_PcbLib:Power_Board_Socket_Conn_1.27mm"
-			(at 89.916 76.2 0)
+		(property "Footprint" "X-MODs_PcbLib:Power_Board_Socket_Conn_1.27mm"
+			(at 90.932 77.47 0)
 			(effects
 				(font
@@
 		)
 		(property "Description" "Power_Board_Socket_Conn_1.27mm"
-			(at 101.092 74.168 0)
+			(at 99.822 75.438 0)
 			(effects
 				(font
@@
 	)
 	(symbol
-		(lib_id "HeepoMind_SchLib:Power_Board_Socket_Conn_1.27mm")
+		(lib_id "X-MODs_SchLib:Power_Board_Socket_Conn_1.27mm")
 		(at 191.77 81.28 0)
 		(unit 3)
@@
 			)
 		)
-		(property "Footprint" "HeepoMind_PcbLib:Power_Board_Socket_Conn_1.27mm"
-			(at 200.914 111.76 0)
+		(property "Footprint" "X-MODs_PcbLib:Power_Board_Socket_Conn_1.27mm"
+			(at 199.898 113.03 0)
 			(effects
 				(font
@@
 		)
 		(property "Description" "Power_Board_Socket_Conn_1.27mm"
-			(at 189.738 109.728 0)
+			(at 191.008 110.998 0)
 			(effects
 				(font
@@
 	)
 	(symbol
-		(lib_id "HeepoMind_SchLib:Power_Board_Header_Conn_2.54mm")
+		(lib_id "X-MODs_SchLib:Power_Board_Header_Conn_2.54mm")
 		(at 160.02 116.84 180)
 		(unit 2)
@@
 			)
 		)
-		(property "Footprint" "HeepoMind_PcbLib:Power_Board_Header_Conn_2.54mm"
-			(at 159.258 118.11 0)
+		(property "Footprint" "X-MODs_PcbLib:Power_Board_Header_Conn_2.54mm"
+			(at 158.242 59.944 0)
 			(effects
 				(font
@@
 	)
 	(symbol
-		(lib_id "HeepoMind_SchLib:Power_Board_Socket_Conn_1.27mm")
+		(lib_id "X-MODs_SchLib:Power_Board_Socket_Conn_1.27mm")
 		(at 99.06 81.28 0)
 		(mirror y)
@@
 			)
 		)
-		(property "Footprint" "HeepoMind_PcbLib:Power_Board_Socket_Conn_1.27mm"
-			(at 89.916 111.76 0)
+		(property "Footprint" "X-MODs_PcbLib:Power_Board_Socket_Conn_1.27mm"
+			(at 90.932 113.03 0)
 			(effects
 				(font
@@
 		)
 		(property "Description" "Power_Board_Socket_Conn_1.27mm"
-			(at 101.092 109.728 0)
-			(effects
-				(font
+			(at 99.822 110.998 0)
+			(effects
+				(font
