File: Module Boards/Analog_Board/[1] Power Regulation & Level Shifting.kicad_sch (KiCad schematic)
At the start: 25 parts, among them U2 TXB0104RUTR, U3 TPS22916CYFPR, U4 TPS7A9401DSCR

Commit message: Routed Analog Board
Parts:
- added C13: 100n 10V, X-MODs_PcbLib:C0402, symbol X-MODs_SchLib:GRM155R71A104JA01D
Connections:
- net +3VA_ADC: now also C13.1
- net GND: now also C13.2
- net FB_PG: now reaches R15.1, R8.2, U4.5 (FB_PG)
Other:
- moved on the sheet: C4, U3
