File: Module Boards/HEEP_Board/[2] Connectors & Flash.kicad_sch (KiCad schematic)
At the start: 16 parts, among them U4 W25Q128JWYIQ

Commit message: Fixed path dependencies and changed library name to X-MODs
Parts:
- C15, C16, C17, C18: footprint HeepoMind_PcbLib:C0402 -> X-MODs_PcbLib:C0402; symbol HeepoMind_SchLib:GRM155R71A104JA01D -> X-MODs_SchLib:GRM155R71A104JA01D
- J1: footprint HeepoMind_PcbLib:HEEP_Board_Castellated_Conn_1.27mm -> X-MODs_PcbLib:HEEP_Board_Castellated_Conn_1.27mm; symbol HeepoMind_SchLib:HEEP_Board_Castellated_Conn_1.27mm -> X-MODs_SchLib:HEEP_Board_Castellated_Conn_1.27mm
- R4, R5, R6, R7: footprint HeepoMind_PcbLib:R0402 -> X-MODs_PcbLib:R0402; symbol HeepoMind_SchLib:CRCW040210K0FKEDHP -> X-MODs_SchLib:CRCW040210K0FKEDHP
- R8, R9: footprint HeepoMind_PcbLib:R0402 -> X-MODs_PcbLib:R0402; symbol HeepoMind_SchLib:CRCW0402100KFKEDC -> X-MODs_SchLib:CRCW0402100KFKEDC
- SW1: footprint HeepoMind_PcbLib:TL1030AF160AQJ -> X-MODs_PcbLib:TL1030AF160AQJ; symbol HeepoMind_SchLib:TL1030AF160AQJ -> X-MODs_SchLib:TL1030AF160AQJ
- U4: footprint HeepoMind_PcbLib:WLCSP-21 -> X-MODs_PcbLib:WLCSP-21; symbol HeepoMind_SchLib:W25Q128JWYIQ -> X-MODs_SchLib:W25Q128JWYIQ
- U5, U6: footprint HeepoMind_PcbLib:X2SON-8 -> X-MODs_PcbLib:X2SON-8; symbol HeepoMind_SchLib:SN74AUP2G08DQER -> X-MODs_SchLib:SN74AUP2G08DQER
- U7: footprint HeepoMind_PcbLib:X2SON-6 -> X-MODs_PcbLib:X2SON-6; symbol HeepoMind_SchLib:SN74AUP1G14DSFR -> X-MODs_SchLib:SN74AUP1G14DSFR

Commit message: Added Memory Board
Other:
- note added: "128 Mbit Flash Memory"
- note removed: "128M-bit Flash Memory"
Changed lines of the file:
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@@
 		)
 	)
-	(text "128M-bit Flash Memory"
+	(text "128 Mbit Flash Memory"
 		(exclude_from_sim no)
 		(at 24.638 24.13 0)
