File: Module_Boards/ADC_Board/ADC_Board.kicad_sch (KiCad schematic)
At the start: 0 parts

Commit message: Fixed bugs. Added comments. Push before changing the ADC
Other:
- company: (none) -> Embedded Systems Laboratory - EPFL
Changed lines of the file:
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@@
 	(generator_version "8.0")
 	(paper "A4")
+	(title_block
+		(rev "1.0")
+		(company "Embedded Systems Laboratory - EPFL")
+		(comment 1 "Author: José Angel Miranda Calero")
+		(comment 2 "Author: Juan Sapriza")
+		(comment 3 "Author: Alejandro López Rodriguez")
+	)
 	(sheet
 		(at 295.91 30.48)

Commit message: Final revision and production files
Other:
- sheet [1] Power Regulation & Level Shifting renamed [1] Power Regulation & Connectors
- sheet [2] ADC & Multiplexer renamed [2] ADC, Multiplexer & Reference
- sheet [1] Power Regulation & Connectors: file [1] Power Regulation & Level Shifting.kicad_sch -> [1] Power Regulation & Connectors.kicad_sch
- sheet [2] ADC, Multiplexer & Reference: file [2] ADC & Multiplexer.kicad_sch -> [2] ADC, Multiplexer & Reference.kicad_sch
Changed lines of the file:
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@@
 			(color 0 0 0 0.0000)
 		)
-		(property "Sheetname" "[1] Power Regulation & Level Shifting"
+		(property "Sheetname" "[1] Power Regulation & Connectors"
 			(at 295.91 29.7684 0)
 			(effects
@@
 			)
 		)
-		(property "Sheetfile" "[1] Power Regulation & Level Shifting.kicad_sch"
+		(property "Sheetfile" "[1] Power Regulation & Connectors.kicad_sch"
 			(at 295.91 45.0346 0)
 			(effects
@@
 			(color 0 0 0 0.0000)
 		)
-		(property "Sheetname" "[2] ADC & Multiplexer"
+		(property "Sheetname" "[2] ADC, Multiplexer & Reference"
 			(at 295.91 50.0884 0)
 			(effects
@@
 			)
 		)
-		(property "Sheetfile" "[2] ADC & Multiplexer.kicad_sch"
+		(property "Sheetfile" "[2] ADC, Multiplexer & Reference.kicad_sch"
 			(at 295.91 65.3546 0)
 			(effects
