File: Module_Boards/ADC_Board/[1] Power Regulation & Connectors.kicad_sch (KiCad schematic)
At the start: 21 parts, among them U3 TPS22916CYFPR, U4 TPS7A9401DSCR

Commit message: Added fabrication panel. Now with latest designs
Parts:
- U4: symbol X-MODs_SchLib:TPS7A9401DSCR -> X-MODs_SchLib:TPS7A9401DSCR; MPN (none) -> TPS7A9401DSCR
Changed lines of the file:
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@@
 	)
 	(symbol
-		(lib_id "X-MODs_SchLib:TPS7A9401DSCR ")
+		(lib_id "X-MODs_SchLib:TPS7A9401DSCR")
 		(at 186.69 40.64 0)
 		(unit 1)
@@
 				(hide yes)
 			)
+		)
+		(property "MPN" "TPS7A9401DSCR"
+			(at 173.99 76.2 0)
+			(effects
+				(font
+					(size 1.27 1.27)
+				)
+				(hide yes)
+			)
