File: Socket_Boards/Memory_Board_Socket/Memory_Board_Socket.kicad_pcb (KiCad board)
At the start: 4 copper layers, 69.3 x 16.3 mm, 18 parts

Commit message: Final revision and production files
Parts:
- added G***: LOGO, LOGO, B.Cu at (180.3, 96.9)
- added G***: LOGO, LOGO, B.Cu at (137.4, 94.4)
- added kibuzzard-66CFCF0D: G***, kibuzzard-66CFCF0D, B.Cu at (180.3, 102.8)
- added kibuzzard-67530B9C: G***, kibuzzard-67530B9C, B.Cu at (137.4, 100.8)
