File: Socket_Boards/Memory_Board_Socket/Memory_Board_Socket.kicad_sch (KiCad schematic)
At the start: 2 parts

Commit message: Final revision and production files
Other:
- moved on the sheet: J1B
Changed lines of the file:
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@@
 	)
 	(junction
-		(at 186.69 99.06)
+		(at 186.69 96.52)
 		(diameter 0)
 		(color 0 0 0 0)
@@
 	(wire
 		(pts
-			(xy 186.69 99.06) (xy 180.34 99.06)
+			(xy 186.69 96.52) (xy 180.34 96.52)
 		)
 		(stroke
@@
 	(wire
 		(pts
+			(xy 193.04 101.6) (xy 180.34 101.6)
+		)
+		(stroke
+			(width 0)
+			(type default)
+		)
+	)
+	(wire
+		(pts
+			(xy 193.04 99.06) (xy 180.34 99.06)
+		)
+		(stroke
+			(width 0)
+			(type default)
+		)
+	)
+	(wire
+		(pts
+			(xy 106.68 93.98) (xy 100.33 93.98)
+		)
+		(stroke
+			(width 0)
+			(type default)
+		)
+	)
+	(wire
+		(pts
+			(xy 106.68 93.98) (xy 106.68 109.22)
+		)
+		(stroke
+			(width 0)
+			(type default)
+		)
+	)
+	(wire
+		(pts
+			(xy 113.03 104.14) (xy 100.33 104.14)
+		)
+		(stroke
+			(width 0)
+			(type default)
+		)
+	)
+	(wire
+		(pts
+			(xy 193.04 91.44) (xy 180.34 91.44)
+		)
+		(stroke
+			(width 0)
+			(type default)
+		)
+	)
+	(wire
+		(pts
+			(xy 113.03 93.98) (xy 106.68 93.98)
+		)
+		(stroke
+			(width 0)
+			(type default)
+		)
+	)
+	(wire
+		(pts
+			(xy 186.69 109.22) (xy 186.69 96.52)
+		)
+		(stroke
+			(width 0)
+			(type default)
+		)
+	)
+	(wire
+		(pts
 			(xy 193.04 93.98) (xy 180.34 93.98)
 		)
@@
 	(wire
 		(pts
-			(xy 193.04 96.52) (xy 180.34 96.52)
-		)
-		(stroke
-			(width 0)
-			(type default)
-		)
-	)
-	(wire
-		(pts
-			(xy 106.68 93.98) (xy 100.33 93.98)
-		)
-		(stroke
-			(width 0)
-			(type default)
-		)
-	)
-	(wire
-		(pts
-			(xy 106.68 93.98) (xy 106.68 109.22)
-		)
-		(stroke
-			(width 0)
-			(type default)
-		)
-	)
-	(wire
-		(pts
-			(xy 113.03 104.14) (xy 100.33 104.14)
+			(xy 106.68 87.63) (xy 106.68 91.44)
 		)
 		(stroke
@@
 	(wire
 		(pts
-			(xy 113.03 93.98) (xy 106.68 93.98)
-		)
-		(stroke
-			(width 0)
-			(type default)
-		)
-	)
-	(wire
-		(pts
-			(xy 193.04 101.6) (xy 180.34 101.6)
-		)
-		(stroke
-			(width 0)
-			(type default)
-		)
-	)
-	(wire
-		(pts
-			(xy 106.68 87.63) (xy 106.68 91.44)
-		)
-		(stroke
-			(width 0)
-			(type default)
-		)
-	)
-	(wire
-		(pts
-			(xy 193.04 91.44) (xy 180.34 91.44)
-		)
-		(stroke
-			(width 0)
-			(type default)
-		)
-	)
-	(wire
-		(pts
 			(xy 113.03 91.44) (xy 106.68 91.44)
 		)
@@
 	(wire
 		(pts
-			(xy 186.69 99.06) (xy 186.69 109.22)
-		)
-		(stroke
-			(width 0)
-			(type default)
-		)
-	)
-	(wire
-		(pts
-			(xy 193.04 99.06) (xy 186.69 99.06)
+			(xy 193.04 96.52) (xy 186.69 96.52)
 		)
 		(stroke
@@
 	(symbol
 		(lib_id "X-MODs_SchLib:Memory_Board_Header_Conn_2.54mm")
-		(at 195.58 88.9 0)
+		(at 195.58 106.68 0)
+		(mirror x)
 		(unit 2)
 		(exclude_from_sim no)
@@
 		(dnp no)
 		(property "Reference" "J2"
-			(at 195.326 87.5029 0)
+			(at 195.326 87.7571 0)
 			(effects
 				(font
@@
 		)
 		(property "Value" "~"
-			(at 218.44 99.06 0)
+			(at 218.44 96.52 0)
 			(effects
 				(font
@@
 		)
 		(property "Footprint" "X-MODs_PcbLib:Memory_Board_Header_Conn_2.54mm"
-			(at 202.946 111.252 0)
+			(at 202.946 84.328 0)
 			(effects
 				(font
@@
 		)
 		(property "Datasheet" ""
-			(at 195.58 88.9 0)
+			(at 195.58 106.68 0)
 			(effects
 				(font
@@
 		)
 		(property "Description" "Analog_Board_Castellated_Conn_1.27mm"
-			(at 196.85 109.474 0)
+			(at 196.85 86.106 0)
 			(effects
 				(font
@@
 		)
 		(property "MPN" ""
-			(at 195.58 88.9 0)
+			(at 195.58 106.68 0)
 			(effects
 				(font
@@
 		(on_board yes)
 		(dnp no)
-		(fields_autoplaced yes)
 		(property "Reference" "#PWR02"
 			(at 186.69 115.57 0)
@@
 	(symbol
 		(lib_id "X-MODs_SchLib:Memory_Board_Socket_Conn_1.27mm")
-		(at 177.8 88.9 0)
-		(mirror y)
+		(at 177.8 106.68 180)
 		(unit 2)
 		(exclude_from_sim no)
@@
 		(dnp no)
 		(property "Reference" "J1"
-			(at 178.308 87.5029 0)
+			(at 178.054 87.7571 0)
 			(effects
 				(font
@@
 		)
 		(property "Value" "~"
-			(at 154.94 99.06 0)
+			(at 154.94 96.52 0)
 			(effects
 				(font
@@
 		)
 		(property "Footprint" "X-MODs_PcbLib:Memory_Board_Socket_Conn_1.27mm"
-			(at 168.402 111.252 0)
+			(at 168.402 84.328 0)
 			(effects
 				(font
@@
 		)
 		(property "Datasheet" ""
-			(at 177.8 88.9 0)
+			(at 177.8 106.68 0)
 			(effects
 				(font
@@
 		)
 		(property "Description" "Analog_Board_Castellated_Conn_1.27mm"
-			(at 176.53 109.474 0)
+			(at 176.53 86.106 0)
 			(effects
 				(font
@@
 		)
 		(property "MPN" ""
-			(at 177.8 88.9 0)
-			(effects
-				(font
+			(at 177.8 106.68 0)
+			(effects
+				(font
