File: Socket_Boards/Power_Board_Socket/Power_Board_Socket.kicad_pcb (KiCad board)
At the start: 4 copper layers, 38 x 47.3 mm, 41 parts

Commit message: Final revision and production files
Parts:
- removed kibuzzard-66CFD049: G***, kibuzzard-66CFD049
- added kibuzzard-67530430: G***, kibuzzard-67530430, B.Cu at (137.0, 130.0)
- J1: footprint X-MODs_PcbLib:Power_Board_Header_Conn_2.54mm -> X-MODs_PcbLib:Power_Board_Socket_Conn_1.27mm
- J2: footprint X-MODs_PcbLib:Power_Board_Socket_Conn_1.27mm -> X-MODs_PcbLib:Power_Board_Header_Conn_2.54mm
Connections:
- net /+1V8 renamed /[1] 1.27 mm Flexypin to 2.54 mm Header Adapter/+1V8
- net /ALRT renamed /[1] 1.27 mm Flexypin to 2.54 mm Header Adapter/ALRT
- net /AVCC renamed /[1] 1.27 mm Flexypin to 2.54 mm Header Adapter/AVCC
- net /CHG_IN renamed /[1] 1.27 mm Flexypin to 2.54 mm Header Adapter/CHG_IN
- net /GPIO0 renamed /[1] 1.27 mm Flexypin to 2.54 mm Header Adapter/GPIO0
- net /GPIO1 renamed /[1] 1.27 mm Flexypin to 2.54 mm Header Adapter/GPIO1
- net /GPIO2 renamed /[1] 1.27 mm Flexypin to 2.54 mm Header Adapter/GPIO2
- net /SCL renamed /[1] 1.27 mm Flexypin to 2.54 mm Header Adapter/SCL
- net /SDA renamed /[1] 1.27 mm Flexypin to 2.54 mm Header Adapter/SDA
- net /VBAT renamed /[1] 1.27 mm Flexypin to 2.54 mm Header Adapter/VBAT
- net /VCORE renamed /[1] 1.27 mm Flexypin to 2.54 mm Header Adapter/VCORE
- net /VIO renamed /[1] 1.27 mm Flexypin to 2.54 mm Header Adapter/VIO
- net /VSYS renamed /[1] 1.27 mm Flexypin to 2.54 mm Header Adapter/VSYS
- net /nIRQ renamed /[1] 1.27 mm Flexypin to 2.54 mm Header Adapter/nIRQ
- net /nRST renamed /[1] 1.27 mm Flexypin to 2.54 mm Header Adapter/nRST
Routing:
- net GND: track 46.5 -> 93.0 mm
- net /[1] 1.27 mm Flexypin to 2.54 mm Header Adapter/GPIO1: track 13.8 -> 16.9 mm
- net /[1] 1.27 mm Flexypin to 2.54 mm Header Adapter/VSYS: track 12.1 -> 15.2 mm
- net /[1] 1.27 mm Flexypin to 2.54 mm Header Adapter/VCORE: track 12.7 -> 15.8 mm
- net /[1] 1.27 mm Flexypin to 2.54 mm Header Adapter/VBAT: track 13.2 -> 16.3 mm
- net /[1] 1.27 mm Flexypin to 2.54 mm Header Adapter/GPIO0: track 13.2 -> 16.3 mm
- net /[1] 1.27 mm Flexypin to 2.54 mm Header Adapter/CHG_IN: track 12.6 -> 15.7 mm
- net /[1] 1.27 mm Flexypin to 2.54 mm Header Adapter/AVCC: track 12.6 -> 15.7 mm
- net /[1] 1.27 mm Flexypin to 2.54 mm Header Adapter/+1V8: track 13.7 -> 16.8 mm
- net nEN: track 27.1 -> 30.2 mm
- net VLDO1: track 24.5 -> 27.6 mm
- net VLDO0: track 18.2 -> 21.3 mm
- net AMUX: track 20.8 -> 23.9 mm
- net /[1] 1.27 mm Flexypin to 2.54 mm Header Adapter/nRST: track 24.2 -> 27.3 mm
- net /[1] 1.27 mm Flexypin to 2.54 mm Header Adapter/nIRQ: track 21.0 -> 24.1 mm
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