File: Module_Boards/CHEEP_Board/CHEEP_Board.kicad_sch (KiCad schematic)
At the start: 0 parts

Commit message: Push with updated readme
Other:
- company: (none) -> Embedded Systems Laboratory - EPFL
Changed lines of the file:
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@@
 	(generator_version "8.0")
 	(paper "A4")
+	(title_block
+		(rev "1.0")
+		(company "Embedded Systems Laboratory - EPFL")
+		(comment 1 "Author: José Angel Miranda Calero")
+		(comment 2 "Author: Juan Sapriza")
+		(comment 3 "Author: Alejandro López Rodriguez")
+	)
 	(sheet
 		(at 302.26 63.5)
