File: Module_Boards/CHEEP_Board/[1] HEEPocrates.kicad_sch (KiCad schematic)
At the start: 20 parts, among them U2 HEEPocrates, U3 SIT1532AC-J5-DCC-32.768D

Commit message: Big push. Fixed the issues that were pending. See github
Parts:
- removed C13: 100n 10V, X-MODs_PcbLib:C0402, symbol X-MODs_SchLib:GRM155R71A104JA01D
- removed R1: 100K, X-MODs_PcbLib:R0402, symbol X-MODs_SchLib:CRCW0402100KFKEDC
- removed U1: ~, X-MODs_PcbLib:X2SON-6, symbol X-MODs_SchLib:SN74AUP1G14DSFR
- added R1: 10K0, X-MODs_PcbLib:R0402, symbol X-MODs_SchLib:CRCW040210K0FKEDHP
- renumbered C14 to C13, U3 to OSC1, U2 to U1
Connections:
- net BOOT_SELECT is gone; now on net BOOT_SEL_EXT: U1.86 (BOOT_SELECT_I)
- net +1V8: now also R1.1
- net BOOT_SEL_EXT: now also R1.2

Commit message: Fixed bugs. Added comments. Push before changing the ADC
Changed lines of the file:
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@@
 				)
 				(justify left)
+				(hide yes)
 			)
 		)

Commit message: Push with updated readme
Other:
- company: (none) -> Embedded Systems Laboratory - EPFL
- title: (none) -> [1] HEEPocrates
Changed lines of the file:
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@@
 	(generator_version "8.0")
 	(paper "A4")
+	(title_block
+		(title "[1] HEEPocrates")
+		(rev "1.0")
+		(company "Embedded Systems Laboratory - EPFL")
+		(comment 1 "Author: José Angel Miranda Calero")
+		(comment 2 "Author: Juan Sapriza")
+		(comment 3 "Author: Alejandro López Rodriguez")
+	)
 	(junction
 		(at 222.25 29.21)
@@
 	(text_box "Boot Procedure:\n	- SPI Flash Load → BOOT_SEL_EXT = 1 (Default)\n	- JTAG		   → BOOT_SEL_EXT = 0 "
 		(exclude_from_sim no)
-		(at 224.79 69.85 0)
+		(at 218.44 69.85 0)
 		(size 58.42 7.62)
 		(stroke
