File: Module_Boards/Memory_Board/Memory_Board.kicad_sch (KiCad schematic)
At the start: 12 parts, among them U1 MX25U12832FZNI02-TR, U2 MX25U25643GZ4I00-T

Commit message: Push with updated readme
Other:
- company: (none) -> Embedded Systems Laboratory - EPFL
- title: (none) -> [1] Flash memories & Connectors
Changed lines of the file:
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@@
 	(generator_version "8.0")
 	(paper "A4")
+	(title_block
+		(title "[1] Flash memories & Connectors")
+		(rev "1.0")
+		(company "Embedded Systems Laboratory - EPFL")
+		(comment 1 "Author: José Angel Miranda Calero")
+		(comment 2 "Author: Juan Sapriza")
+		(comment 3 "Author: Alejandro López Rodriguez")
+	)
 	(junction
 		(at 58.42 124.46)
