File: Module_Boards/Power_Board/[1] Battery Gauge & Connectors.kicad_sch (KiCad schematic)
At the start: 6 parts, among them U1 MAX17262REWL+T

Commit message: Fixed bugs. Added comments. Push before changing the ADC
Parts:
- C2: symbol X-MODs_SchLib:GRM155R60J474KE19 -> X-MODs_SchLib:GRM155R60J474KE19D; MPN (none) -> GRM155R60J474KE19D
Other:
- note added: "Battery Fuel Gauge"
- note removed: "Battery Gauge"
Changed lines of the file:
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@@
 	(title_block
 		(title "[2] Battery Gauge & Connectors")
-		(rev "0.1")
+		(rev "1.0")
 		(company "Embedded Systems Laboratory - EPFL")
+		(comment 1 "Author: José Angel Miranda Calero")
+		(comment 2 "Author: Juan Sapriza")
+		(comment 3 "Author: Alejandro López Rodriguez")
 	)
 	(junction
@@
 		)
 	)
-	(text_box "ALRT Pin - Fuel-gauge alerts (Open Collector):\n• DEFAULT: 0 Ohm Resistor to GND (Disabled)\n• ALT: Pull-up Resistor to +1V8\n\n"
+	(text_box "The MAX17262 has an ALERT pin (ALRT) that goes low if \nprogrammable events happens (voltage/current exceeds X, etc)\n• WHEN NOT USED: 0 Ohm resistor to GND (Default case)\n• ENABLED: Remove R2 and populate R1 (10 kOhm)\n\nSimilarly, it has a thermistor input (TH), which has been disabled since LiPo batteries\ncome with external protection. TH Pin can be used for battery insertion detection.\n"
 		(exclude_from_sim no)
-		(at 58.42 62.23 0)
-		(size 50.8 7.62)
+		(at 41.91 53.34 0)
+		(size 90.17 16.51)
 		(stroke
 			(width 0)
@@
 		)
 	)
-	(text "Battery Gauge"
+	(text "Battery Fuel Gauge"
 		(exclude_from_sim no)
 		(at 34.798 46.99 0)
@@
 	)
 	(symbol
-		(lib_id "X-MODs_SchLib:GRM155R60J474KE19")
+		(lib_id "X-MODs_SchLib:GRM155R60J474KE19D")
 		(at 100.33 106.68 270)
 		(unit 1)
@@
 		)
 		(property "Footprint" "X-MODs_PcbLib:C0402"
-			(at 92.202 80.264 0)
+			(at 92.202 79.248 0)
 			(effects
 				(font
@@
 		(property "Description" "Multilayer Ceramic Capacitors MLCC - SMD/SMT 0.47 uF 6.3 VDC 10% 0402 X5R"
 			(at 96.266 108.458 0)
+			(effects
+				(font
+					(size 1.27 1.27)
+				)
+				(hide yes)
+			)
+		)
+		(property "MPN" "GRM155R60J474KE19D"
+			(at 90.17 79.248 0)
 			(effects
 				(font
@@
 		(dnp no)
 		(property "Reference" "U1"
-			(at 83.185 73.66 0)
+			(at 73.279 75.438 0)
 			(effects
 				(font
@@
 		)
 		(property "Value" "MAX17262REWL+T"
-			(at 83.185 76.2 0)
-			(effects
-				(font
+			(at 80.645 77.47 0)
+			(effects
+				(font

Commit message: Push with updated readme
Other:
- moved on the sheet: C1, C2, R1, R2, U1
